File: Kicad/tof_sensor.kicad_pcb (KiCad board)
At the start: 2 copper layers, 86.4 x 45.7 mm, 57 parts, among them J1 Conn_01x06_Male, J2 Conn_01x05, Q1 BSH202,215, SW1 SW_DIP_x03, U1 MIC5504-2.8YM5, U2 PIC24FJ64GA002, U3 VL53L0X, U4 VL53L0X, U5 PCA9306

Commit message: Updated D1 Footprint
Changed from 1206 to SOD-323
Parts:
- D1: footprint Diodes_SMD:D_1206 -> Diode_SMD:D_SOD-323_HandSoldering
Changed lines of the file:
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@@
     (thickness 1.6)
     (drawings 68)
-    (tracks 420)
+    (tracks 422)
     (zones 0)
     (modules 57)
@@
     (zone_45_only no)
     (trace_min 0.2)
+    (segment_width 0.2)
+    (edge_width 0.05)
     (via_size 0.8)
     (via_drill 0.4)
@@
     (uvia_min_size 0.2)
     (uvia_min_drill 0.1)
-    (edge_width 0.05)
-    (segment_width 0.2)
     (pcb_text_width 0.3)
     (pcb_text_size 1.5 1.5)
@@
     )
   )
-  (module Diodes_SMD:D_1206 (layer F.Cu)
-    (at 146.05 72.39 180)
-    (descr "Diode SMD 1206, reflow soldering http://datasheets.avx.com/schottky.pdf")
-    (tags "Diode 1206")
-    (attr smd)
-    (fp_text reference D1 (at 0 -1.905) (layer F.SilkS)
-      (effects (font (size 1 1) (thickness 0.15)))
-    )
-    (fp_text value D_Schottky (at 0 1.9) (layer F.Fab)
-      (effects (font (size 1 1) (thickness 0.15)))
-    )
-    (fp_text user %R (at 0 -1.8) (layer F.Fab)
-      (effects (font (size 1 1) (thickness 0.15)))
-    )
-    (fp_line (start -0.254 -0.254) (end -0.254 0.254) (layer F.Fab) (width 0.1))
-    (fp_line (start 0.127 0) (end 0.381 0) (layer F.Fab) (width 0.1))
-    (fp_line (start -0.254 0) (end -0.508 0) (layer F.Fab) (width 0.1))
-    (fp_line (start 0.127 0.254) (end -0.254 0) (layer F.Fab) (width 0.1))
-    (fp_line (start 0.127 -0.254) (end 0.127 0.254) (layer F.Fab) (width 0.1))
-    (fp_line (start -0.254 0) (end 0.127 -0.254) (layer F.Fab) (width 0.1))
-    (fp_line (start -2.2 -1.06) (end -2.2 1.06) (layer F.SilkS) (width 0.12))
-    (fp_line (start -1.7 0.95) (end -1.7 -0.95) (layer F.Fab) (width 0.1))
-    (fp_line (start 1.7 0.95) (end -1.7 0.95) (layer F.Fab) (width 0.1))
-    (fp_line (start 1.7 -0.95) (end 1.7 0.95) (layer F.Fab) (width 0.1))
-    (fp_line (start -1.7 -0.95) (end 1.7 -0.95) (layer F.Fab) (width 0.1))
-    (fp_line (start -2.3 -1.16) (end 2.3 -1.16) (layer F.CrtYd) (width 0.05))
-    (fp_line (start -2.3 1.16) (end 2.3 1.16) (layer F.CrtYd) (width 0.05))
-    (fp_line (start -2.3 -1.16) (end -2.3 1.16) (layer F.CrtYd) (width 0.05))
-    (fp_line (start 2.3 -1.16) (end 2.3 1.16) (layer F.CrtYd) (width 0.05))
-    (fp_line (start 1 -1.06) (end -2.2 -1.06) (layer F.SilkS) (width 0.12))
-    (fp_line (start -2.2 1.06) (end 1 1.06) (layer F.SilkS) (width 0.12))
-    (pad 1 smd rect (at -1.5 0 180) (size 1 1.6) (layers F.Cu F.Paste F.Mask)
-      (net 5 /Vpp))
-    (pad 2 smd rect (at 1.5 0 180) (size 1 1.6) (layers F.Cu F.Paste F.Mask)
-      (net 24 "Net-(C10-Pad1)"))
-    (model ${KISYS3DMOD}/Diodes_SMD.3dshapes/D_1206.wrl
-      (at (xyz 0 0 0))
-      (scale (xyz 1 1 1))
-      (rotate (xyz 0 0 0))
-    )
-  )
   (module Capacitors_SMD:C_1206_HandSoldering (layer F.Cu)
     (at 167.64 82.55)
@@
       (net 2 GND))
     (model Capacitors_SMD.3dshapes/C_1206.wrl
+      (at (xyz 0 0 0))
+      (scale (xyz 1 1 1))
+      (rotate (xyz 0 0 0))
+    )
+  )
+  (module Diode_SMD:D_SOD-323_HandSoldering (layer F.Cu)
+    (at 146.05 72.39 180)
+    (descr SOD-323)
+    (tags SOD-323)
+    (attr smd)
+    (fp_text reference D1 (at 0 -1.85 180) (layer F.SilkS)
+      (effects (font (size 1 1) (thickness 0.15)))
+    )
+    (fp_text value D_Schottky (at 0.1 1.9 180) (layer F.Fab)
+      (effects (font (size 1 1) (thickness 0.15)))
+    )
+    (fp_text user %R (at 0 -1.85 180) (layer F.Fab)
+      (effects (font (size 1 1) (thickness 0.15)))
+    )
+    (fp_line (start -1.9 -0.85) (end -1.9 0.85) (layer F.SilkS) (width 0.12))
+    (fp_line (start 0.2 0) (end 0.45 0) (layer F.Fab) (width 0.1))
+    (fp_line (start 0.2 0.35) (end -0.3 0) (layer F.Fab) (width 0.1))
+    (fp_line (start 0.2 -0.35) (end 0.2 0.35) (layer F.Fab) (width 0.1))
+    (fp_line (start -0.3 0) (end 0.2 -0.35) (layer F.Fab) (width 0.1))
+    (fp_line (start -0.3 0) (end -0.5 0) (layer F.Fab) (width 0.1))
+    (fp_line (start -0.3 -0.35) (end -0.3 0.35) (layer F.Fab) (width 0.1))
+    (fp_line (start -0.9 0.7) (end -0.9 -0.7) (layer F.Fab) (width 0.1))
+    (fp_line (start 0.9 0.7) (end -0.9 0.7) (layer F.Fab) (width 0.1))
+    (fp_line (start 0.9 -0.7) (end 0.9 0.7) (layer F.Fab) (width 0.1))
+    (fp_line (start -0.9 -0.7) (end 0.9 -0.7) (layer F.Fab) (width 0.1))
+    (fp_line (start -2 -0.95) (end 2 -0.95) (layer F.CrtYd) (width 0.05))
+    (fp_line (start 2 -0.95) (end 2 0.95) (layer F.CrtYd) (width 0.05))
+    (fp_line (start -2 0.95) (end 2 0.95) (layer F.CrtYd) (width 0.05))
+    (fp_line (start -2 -0.95) (end -2 0.95) (layer F.CrtYd) (width 0.05))
+    (fp_line (start -1.9 0.85) (end 1.25 0.85) (layer F.SilkS) (width 0.12))
+    (fp_line (start -1.9 -0.85) (end 1.25 -0.85) (layer F.SilkS) (width 0.12))
+    (pad 1 smd rect (at -1.25 0 180) (size 1 1) (layers F.Cu F.Paste F.Mask)
+      (net 5 /Vpp))
+    (pad 2 smd rect (at 1.25 0 180) (size 1 1) (layers F.Cu F.Paste F.Mask)
+      (net 24 "Net-(C10-Pad1)"))
+    (model ${KISYS3DMOD}/Diode_SMD.3dshapes/D_SOD-323.wrl
       (at (xyz 0 0 0))
       (scale (xyz 1 1 1))
@@
   (segment (start 136.43 64.77) (end 136.525 64.865) (width 0.25) (layer F.Cu) (net 4) (status 30))
   (segment (start 132.51 68.875) (end 132.51 69.525) (width 0.25) (layer F.Cu) (net 4))
-  (segment (start 147.55 72.39) (end 148.59 72.39) (width 0.25) (layer F.Cu) (net 5) (status 10))
   (segment (start 149.225 73.025) (end 151.6888 73.025) (width 0.25) (layer F.Cu) (net 5) (status 20))
-  (segment (start 148.59 72.39) (end 149.225 73.025) (width 0.25) (layer F.Cu) (net 5))
   (via (at 163.83 74.93) (size 0.8) (drill 0.4) (layers F.Cu B.Cu) (net 5))
   (segment (start 163.83 74.93) (end 159.385 74.93) (width 0.25) (layer B.Cu) (net 5))
@@
   (segment (start 187.96 68.58) (end 186.69 67.31) (width 0.25) (layer F.Cu) (net 5))
   (segment (start 186.69 67.31) (end 177.165 67.31) (width 0.25) (layer F.Cu) (net 5))
+  (segment (start 148.59 72.39) (end 149.225 73.025) (width 0.25) (layer F.Cu) (net 5))
+  (segment (start 147.3 72.39) (end 148.59 72.39) (width 0.25) (layer F.Cu) (net 5))
   (segment (start 165.64 82.55) (end 163.83 82.55) (width 0.25) (layer F.Cu) (net 6) (status 10))
   (segment (start 163.195 83.185) (end 160.7312 83.185) (width 0.25) (layer F.Cu) (net 6) (status 20))
@@
   (segment (start 141.7 72.39) (end 142.24 71.85) (width 0.25) (layer F.Cu) (net 24) (status 30))
   (segment (start 142.24 71.85) (end 142.24 72.39) (width 0.25) (layer F.Cu) (net 24) (status 30))
-  (segment (start 142.24 72.39) (end 144.55 72.39) (width 0.25) (layer F.Cu) (net 24) (status 30))
   (segment (start 144.55 69.985) (end 144.685 69.85) (width 0.25) (layer F.Cu) (net 24) (status 30))
-  (segment (start 144.55 72.39) (end 144.55 69.985) (width 0.25) (layer F.Cu) (net 24) (status 30))
+  (segment (start 144.8 69.965) (end 144.685 69.85) (width 0.25) (layer F.Cu) (net 24))
+  (segment (start 144.8 72.39) (end 144.8 69.965) (width 0.25) (layer F.Cu) (net 24))
+  (segment (start 144.705 72.485) (end 144.8 72.39) (width 0.25) (layer F.Cu) (net 24))
+  (segment (start 142.24 72.485) (end 144.705 72.485) (width 0.25) (layer F.Cu) (net 24))
   (segment (start 123.19 65.945) (end 123.19 64.695) (width 0.25) (layer F.Cu) (net 35))
   (segment (start 123.19 64.695) (end 123.19 64.262) (width 0.25) (layer F.Cu) (net 35))

Commit message: Updated PCB layout
Parts:
- removed REF**: Symbol_GNU-Logo_SilkscreenTop, Symbols:Symbol_GNU-Logo_SilkscreenTop
- removed REF** (x4): MountingHole_2.2mm_M2_Pad_Via, Mounting_Holes:MountingHole_2.2mm_M2_Pad_Via
- R15: value 330R -> 47R
- U2: footprint footprints:PIC24FJ64GA002-E&slash_SO -> Package_SO:SOIC-28W_7.5x17.9mm_P1.27mm
